File: kicad/07/07.kicad_pcb (KiCad board)
At the start: 2 copper layers, 66 x 25.4 mm, 10 parts, among them J1 ISP, M1 ATTINY45SI, SW1 6MM_SWITCH6MM_SWITCH

Commit message: good ones
Parts:
- removed J1: ISP, fab-2X03
- added M2: AVRISPSMD, fab-2X03SMD, F.Cu at (340.4, 323.9)
- moved FTDI1 6.35 mm to (388.6, 323.9)
- moved R2 4.78 mm to (379.9, 326.4)
Routing:
- net Net-(C1-Pad2): track 82.6 -> 97.6 mm
- net Net-(FTDI1-Pad5): track 64.0 -> 51.0 mm
- net Net-(M1-Pad7): track 52.4 -> 41.5 mm
- net Net-(C1-Pad1): track 110.5 -> 119.9 mm
- net Net-(M1-Pad5): track 29.1 -> 22.7 mm
- net Net-(M1-Pad1): track 31.4 -> 25.2 mm
- net Net-(FTDI1-Pad4): track 9.52 -> 7.85 mm
Other:
- board size 66 x 25.4 mm -> 62.2 x 27.9 mm
- net class Default: trace_width 0.4 -> 0.8
- rule trace_min: 0.4 -> 0.8
